Commit message: checkin moveit-config, kuka node, rviz plugins

File: kuka_kr10_support/urdf/kr10r1100sixx_macro.xacro (robot description, xacro)
@@ -3,5 +3,18 @@
   <xacro:include filename="$(find kuka_resources)/urdf/common_constants.xacro"/>
   <xacro:include filename="$(find kuka_resources)/urdf/common_materials.xacro"/>
+  <xacro:property name="baseheight" value=".400" />
+  <xacro:property name="link1height" value="0"/>
+  <xacro:property name="link2height" value=".56" />
+  <xacro:property name="link3length" value=".035"/>
+  <xacro:property name="link4length" value=".515"/>
+  <xacro:property name="link5length" value=".01" />
+  <xacro:property name="link6length" value=".08" />
+  <xacro:property name="PI" value="3.1415926535897931"/>
   <xacro:macro name="kuka_kr10r1100sixx" params="prefix">
+    <link name="world"/>
+    <joint name="fixed" type="fixed">
+      <parent link="world"/>
+      <child link="${prefix}base_link"/>
+    </joint>
     <link name="${prefix}base_link">
       <visual>
@@ -18,4 +31,12 @@
         </geometry>
       </collision>
+      <inertial>
+        <origin xyz="0 0 0" rpy="0 0 0"/>
+        <mass value="13.5"/>
+	<inertia
+	    ixx="0.27" ixy="0" ixz="-0.07"
+	    iyy="0.36" iyz="0"
+	    izz="0.17"/>
+      </inertial>
     </link>
     <link name="${prefix}link_1">
@@ -33,4 +54,12 @@
         </geometry>
       </collision>
+      <inertial>
+        <origin xyz="0 0 0" rpy="0 0 0"/>
+        <mass value="11.4"/>
+	<inertia
+	    ixx="0.15" ixy="0.0" ixz="0"
+	    iyy="0.13" iyz="0"
+	    izz="0.09"/>
+      </inertial>
     </link>
     <link name="${prefix}link_2">
@@ -48,4 +77,12 @@
         </geometry>
       </collision>
+      <inertial>
+        <origin xyz="0 0 0" rpy="0 0 0"/>
+        <mass value="20.63"/>
+	<inertia
+	    ixx="0.11" ixy="-0.02" ixz="0"
+	    iyy="2.65" iyz="0"
+	    izz="2.67"/>
+      </inertial>
     </link>
     <link name="${prefix}link_3">
@@ -63,4 +100,12 @@
         </geometry>
       </collision>
+      <inertial>
+        <origin xyz="0 0 0" rpy="0 0 0"/>
+        <mass value="3.06"/>
+	<inertia
+	    ixx="0.01" ixy="0" ixz="0"
+	    iyy="0.01" iyz="0"
+	    izz="0.01"/>
+      </inertial>
     </link>
     <link name="${prefix}link_4">
@@ -78,4 +123,12 @@
         </geometry>
       </collision>
+      <inertial>
+        <origin xyz="0 0 0" rpy="0 0 0"/>
+        <mass value="5.09"/>
+	<inertia
+	    ixx="0.01" ixy="0" ixz="0.01"
+	    iyy="0.61" iyz="0"
+	    izz="0.61"/>
+      </inertial>
     </link>
     <link name="${prefix}link_5">
@@ -93,4 +146,12 @@
         </geometry>
       </collision>
+      <inertial>
+        <origin xyz="0 0 0" rpy="0 0 0"/>
+        <mass value=".52"/>
+	<inertia
+	    ixx="0" ixy="0" ixz="0"
+	    iyy="0" iyz="0"
+	    izz="0"/>
+      </inertial>
     </link>
     <link name="${prefix}link_6">
@@ -108,4 +169,12 @@
         </geometry>
       </collision>
+      <inertial>
+        <origin xyz="0 0 0" rpy="0 0 0"/>
+        <mass value="0.2"/>
+	<inertia
+	    ixx="0" ixy="0" ixz="0"
+	    iyy="0" iyz="0"
+	    izz="0"/>
+      </inertial>
     </link>
     <!-- This frame corresponds to the $FLANGE coordinate system in KUKA KRC controllers. -->
