Commit message: WIP refer #3, #25, urdf end effector made right.

File: kuka_kr6r900_with_hotend/kr6r900sixx_with_hotend/urdf/kr6r900sixx_with_hotend.urdf (robot description, URDF)
Before this commit: robot kr6r900sixx_with_hotend, 11 links, 10 joints
Joints:
- joint hotend_to_tip: origin xyz=0.15098 0.000655 0.115553 rpy=0 0.78526059641 0 -> xyz=0.15098 0.000655 0.115553 rpy=0 1.5708 0

File: kuka_kr6r900_with_hotend/kr6r900sixx_with_hotend/urdf/kr6r900sixx_with_hotend.xacro (robot description, xacro)
@@ -49,5 +49,5 @@
 		<parent link="hotend"/>
 		<child link="tool_tip"/>
-		<origin xyz="0.15098 0.000655 0.115553" rpy="0 0.78526059641 0" />
+		<origin xyz="0.15098 0.000655 0.115553" rpy="0 1.5708 0" />
 	</joint>
 </robot>
