Commit message: workspace collision model added.

File: framefab_robot/kuka/framefab_kr6_r900/framefab_kr6_r900_support/urdf/kr6_r900_workspace.urdf (robot description, URDF)
Before this commit: robot kr6_r900_workspace, 13 links, 12 joints
Links:
- added link workspace_base_link
- added link workspace_objects; collision mesh filename=package://framefab_kr6_r900_support/meshes/collision/MIT_3-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
Joints:
- added joint workspace_baselink_to_objects: type fixed, parent workspace_base_link, child workspace_objects, origin xyz=0 0 0 rpy=0 0 0
- added joint world_to_workspace: type fixed, parent world_frame, child workspace_base_link, origin xyz=0 0 0 rpy=0 0 0
- joint eef_to_hotend_tcp_frame: origin xyz=0.15045 0.000282 0.121277 rpy=0 1.57079632679 0 -> xyz=0.15045 0.000283 0.121277 rpy=0 1.57079632679 0

File: framefab_robot/kuka/framefab_kr6_r900/framefab_kr6_r900_support/urdf/kr6_r900_workspace.xacro (robot description, xacro)
@@ -3,4 +3,5 @@
   <xacro:include filename="$(find kuka_kr6_support)/urdf/kr6r900sixx_macro.xacro"/>
   <xacro:include filename="$(find asw_end_effector)/urdf/asw_eef_macro.xacro"/>
+	<xacro:include filename="$(find framefab_kr6_r900_support)/urdf/mit_3-412_workspace_micro.xacro"/>
   <link name="world_frame"/>
   <!-- instantiating arm  -->
@@ -8,4 +9,5 @@
   <!-- instantiating end effector  -->
   <xacro:asw_eef_definition prefix=""/>
+	<xacro:mit_workspace prefix=""/>
   <!-- Attach the end effector to the end of the robot arm (tool0) -->
   <joint name="link_t_to_eef" type="fixed">
@@ -20,3 +22,8 @@
     <origin xyz="0 0 0" rpy="0 0 0"/>
   </joint>
+  <joint name="world_to_workspace" type="fixed">
+    <parent link="world_frame"/>
+    <child link="workspace_base_link"/>
+    <origin xyz="0 0 0" rpy="0 0 0"/>
+  </joint>
 </robot>

Commit message: workspace visual model added.

File: framefab_robot/kuka/framefab_kr6_r900/framefab_kr6_r900_support/urdf/kr6_r900_workspace.urdf (robot description, URDF)
Before this commit: robot kr6_r900_workspace, 15 links, 14 joints
Links:
- link workspace_objects: geometry collision mesh filename=package://framefab_kr6_r900_support/meshes/collision/MIT_3-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; visual mesh filename=package://framefab_kr6_r900_support/meshes/visual/MIT_3-412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

File: framefab_robot/kuka/framefab_kr6_r900/framefab_kr6_r900_support/urdf/mit_3-412_workspace_micro.xacro (robot description, xacro)
@@ -7,4 +7,12 @@
 	<link name="${prefix}workspace_base_link" />
   <link name="${prefix}workspace_objects">
+    <visual>
+      <geometry>
+				<mesh filename="package://framefab_kr6_r900_support/meshes/visual/MIT_3-412_workspace_full.stl"/>
+      </geometry>
+      <material name="grey">
+        <color rgba="0.5 0.5 0.5 1.0"/>
+      </material>
+    </visual>
     <collision>
       <geometry>

Commit message: take off working env objs and collision objs. ik sol not found.

File: framefab_robot/kuka/framefab_kr6_r900/framefab_kr6_r900_support/urdf/kr6_r900_workspace.urdf (robot description, URDF)
Before this commit: robot kr6_r900_workspace, 15 links, 14 joints
Links:
- removed link workspace_base_link
- removed link workspace_objects
Joints:
- removed joint workspace_baselink_to_objects
- removed joint world_to_workspace

File: framefab_robot/kuka/framefab_kr6_r900/framefab_kr6_r900_support/urdf/kr6_r900_workspace.xacro (robot description, xacro)
@@ -3,5 +3,5 @@
   <xacro:include filename="$(find kuka_kr6_support)/urdf/kr6r900sixx_macro.xacro"/>
   <xacro:include filename="$(find asw_end_effector)/urdf/asw_eef_macro.xacro"/>
-	<xacro:include filename="$(find framefab_kr6_r900_support)/urdf/mit_3-412_workspace_micro.xacro"/>
+<!--	<xacro:include filename="$(find framefab_kr6_r900_support)/urdf/mit_3-412_workspace_micro.xacro"/>-->
   <link name="world_frame"/>
   <!-- instantiating arm  -->
@@ -9,5 +9,5 @@
   <!-- instantiating end effector  -->
   <xacro:asw_eef_definition prefix=""/>
-	<xacro:mit_workspace prefix=""/>
+<!--	<xacro:mit_workspace prefix=""/>-->
   <!-- Attach the end effector to the end of the robot arm (tool0) -->
   <joint name="link_t_to_eef" type="fixed">
@@ -22,8 +22,8 @@
     <origin xyz="0 0 0" rpy="0 0 0"/>
   </joint>
-  <joint name="world_to_workspace" type="fixed">
-    <parent link="world_frame"/>
-    <child link="workspace_base_link"/>
-    <origin xyz="0 0 0" rpy="0 0 0"/>
-  </joint>
+<!--  <joint name="world_to_workspace" type="fixed">-->
+<!--    <parent link="world_frame"/>-->
+<!--    <child link="workspace_base_link"/>-->
+<!--    <origin xyz="0 0 0" rpy="0 0 0"/>-->
+<!--  </joint>-->
 </robot>
