Commit message: material feeder added in robot model. Collision model working for planning, refer #68.

File: framefab_robot/kuka/framefab_kr6_r900/framefab_kr6_r900_support/urdf/kr6_r900_workspace.xacro (robot description, xacro)
@@ -1,29 +1,41 @@
 <?xml version="1.0" ?>
 <robot name="kr6_r900_workspace" xmlns:xacro="http://ros.org/wiki/xacro">
-  <xacro:include filename="$(find kuka_kr6_support)/urdf/kr6r900sixx_macro.xacro"/>
-  <xacro:include filename="$(find asw_end_effector)/urdf/asw_eef_macro.xacro"/>
+ 	<xacro:include filename="$(find kuka_kr6_support)/urdf/kr6r900sixx_macro.xacro"/>
+	<xacro:include filename="$(find asw_end_effector)/urdf/asw_eef_macro.xacro"/>
+	<xacro:include filename="$(find asw_material_feeder)/urdf/asw_material_feeder_macro.xacro"/>
 	<xacro:include filename="$(find framefab_kr6_r900_support)/urdf/mit_3-412_workspace_micro.xacro"/>
-  <link name="world_frame"/>
-  <!-- instantiating arm  -->
-  <xacro:kuka_kr6r900sixx prefix=""/>
-  <!-- instantiating end effector  -->
-  <xacro:asw_eef_definition prefix=""/>
+	<xacro:property name="link4_mount_base_x" value="0.06762"/>
+	<xacro:property name="link4_mount_base_y" value="0.0"/>
+	<xacro:property name="link4_mount_base_z" value="0.0575"/>
+	<link name="world_frame"/>
+	<!-- instantiating arm  -->
+	<xacro:kuka_kr6r900sixx prefix=""/>
+	<!-- instantiating end effector  -->
+	<xacro:asw_eef_definition prefix=""/>
+	<!-- instantiating material feeder  -->
+	<xacro:asw_material_feeder_definition prefix=""/>
 	<xacro:mit_workspace prefix=""/>
-  <!-- Attach the end effector to the end of the robot arm (tool0) -->
-  <joint name="link_t_to_eef" type="fixed">
-    <parent link="tool0"/>
-    <child link="eef_frame"/>
-    <origin xyz="0 0 0" rpy="0 0 0"/>
-  </joint>
-  <!-- start of arm-workcell joint definitions -->
-  <joint name="world_to_base" type="fixed">
-    <parent link="world_frame"/>
-    <child link="base_link"/>
-    <origin xyz="0 0 0" rpy="0 0 0"/>
-  </joint>
-  <joint name="world_to_workspace" type="fixed">
-    <parent link="world_frame"/>
-    <child link="workspace_base_link"/>
-    <origin xyz="0 0 0" rpy="0 0 0"/>
-  </joint>
+	<!-- Attach the end effector to the end of the robot arm (tool0) -->
+	<joint name="link_t_to_eef" type="fixed">
+		<parent link="tool0"/>
+		<child link="eef_frame"/>
+		<origin xyz="0 0 0" rpy="0 0 0"/>
+	</joint>
+	<!-- Attach the material feeder to the link4 mount point of the robot arm -->
+    <joint name="link_4_to_link_4_mount_point" type="fixed">
+        <parent link="link_4"/>
+        <child link="link_4_mount_point"/>
+        <origin xyz="${link4_mount_base_x} ${link4_mount_base_y} ${link4_mount_base_z}" rpy="0 0 0"/>
+    </joint>
+	<!-- start of arm-workcell joint definitions -->
+	<joint name="world_to_base" type="fixed">
+		<parent link="world_frame"/>
+		<child link="base_link"/>
+		<origin xyz="0 0 0" rpy="0 0 0"/>
+	</joint>
+	<joint name="world_to_workspace" type="fixed">
+		<parent link="world_frame"/>
+		<child link="workspace_base_link"/>
+		<origin xyz="0 0 0" rpy="0 0 0"/>
+	</joint>
 </robot>

File: framefab_robot/kuka/framefab_kr6_r900/framefab_kr6_r900_support/urdf/mit_3-412_workspace_micro.xacro (robot description, xacro)
@@ -4,26 +4,26 @@
 <!-- Origin is at the robot (kuka_kr6r900) mounting location -->
 <robot xmlns:xacro="http://ros.org/wiki/xacro">
-	<xacro:macro name="mit_workspace" params="prefix">
-	<link name="${prefix}workspace_base_link" />
-  <link name="${prefix}workspace_objects">
-    <visual>
-      <geometry>
-				<mesh filename="package://framefab_kr6_r900_support/meshes/visual/MIT_3-412_workspace_full.stl"/>
-      </geometry>
-      <material name="grey">
-        <color rgba="0.5 0.5 0.5 1.0"/>
-      </material>
-    </visual>
-    <collision>
-      <geometry>
-				<mesh filename="package://framefab_kr6_r900_support/meshes/collision/MIT_3-412_workspace_simplified.stl"/>
-      </geometry>
-    </collision>
-  </link>
-  <joint name="${prefix}workspace_baselink_to_objects" type="fixed">
-    <parent link="${prefix}workspace_base_link"/>
-    <child link="${prefix}workspace_objects"/>
-    <origin xyz="0 0 0" rpy="0 0 0"/>
-  </joint>
-  </xacro:macro>
+<xacro:macro name="mit_workspace" params="prefix">
+<link name="${prefix}workspace_base_link"/>
+<link name="${prefix}workspace_objects">
+<visual>
+	<geometry>
+		<mesh filename="package://framefab_kr6_r900_support/meshes/visual/MIT_3-412_workspace_full.stl"/>
+	</geometry>
+	<material name="grey">
+    	<color rgba="0.5 0.5 0.5 1.0"/>
+	</material>
+</visual>
+<collision>
+	<geometry>
+		<mesh filename="package://framefab_kr6_r900_support/meshes/collision/MIT_3-412_workspace_simplified.stl"/>
+	</geometry>
+</collision>
+</link>
+<joint name="${prefix}workspace_baselink_to_objects" type="fixed">
+	<parent link="${prefix}workspace_base_link"/>
+	<child link="${prefix}workspace_objects"/>
+	<origin xyz="0 0 0" rpy="0 0 0"/>
+</joint>
+</xacro:macro>
 </robot>
