Commit message: irb2400 w linear track compiled as dae. error in iffast generation "6dof needed".

File: framefab_robot/abb/framefab_irb2400/framefab_irb2400_support/urdf/irb2400_with_linear_track.urdf (robot description, URDF)
Before this commit: robot irb2400_workspace, 17 links, 16 joints
Links:
- removed link demo_cell_base_link
- removed link eef_frame
- removed link hotend_tool
- removed link tcp_frame
- removed link tmp_tcp_frame
- removed link workcell_bounds
- removed link world_frame
Joints:
- removed joint cell_base_to_bounds
- removed joint cell_base_to_rail
- removed joint eef_frame_to_hotend_tool
- removed joint eef_to_hotend_tcp_frame
- removed joint link_t_to_eef
- removed joint tmp_to_tcp_frame
- removed joint world_to_demo_cell

File: framefab_robot/abb/framefab_irb2400/framefab_irb2400_support/urdf/irb2400_with_linear_track_workspace.xacro (robot description, xacro)
@@ -5,13 +5,17 @@
 	<!--end effector-->
 	<xacro:include filename="$(find asw_end_effector)/urdf/asw_eef_macro.xacro"/>
-	<!--linear track and other setups in the workcell-->
-	<xacro:include filename="$(find framefab_irb2400_support)/urdf/ucla_linear_track_demo_cell_macro.xacro"/>
+	<!--linear track setup-->
+	<xacro:include filename="$(find framefab_irb2400_support)/urdf/simple_linear_track_macro.xacro"/>
+	<!--workcell setup-->
+	<xacro:include filename="$(find framefab_irb2400_support)/urdf/simple_linear_track_demo_cell_macro.xacro"/>
   <link name="world_frame"/>
   <!-- instantiating arm  -->
   <xacro:abb_irb2400 prefix=""/>
   <!-- instantiating end effector  -->
-  <xacro:asw_eef_definition  prefix=""/>
-  <!-- linear track and workcell  -->
-  <xacro:ucla_linear_track_demo_cell  prefix=""/>
+  <xacro:asw_eef_definition prefix=""/>
+	<!-- linear track  -->
+  <xacro:simple_linear_track prefix=""/>
+  <!-- workcell  -->
+  <xacro:simple_linear_track_demo_cell prefix=""/>
 	<!-- Attach the end effector to the end of the robot arm (tool0) -->
 	<joint name="link_t_to_eef" type="fixed">

File: framefab_robot/abb/framefab_irb2400/framefab_irb2400_support/urdf/simple_linear_track_demo_cell_macro.xacro (robot description, xacro)
@@ -1,6 +1,4 @@
 <?xml version="1.0" ?>
-<!--Generates a urdf from the macro in kr210_macro.xacro -->
 <robot xmlns:xacro="http://ros.org/wiki/xacro">
-<xacro:property name="rail_cross_section" value="0.1"/>
 <xacro:property name="workcell_width" value="5.0"/>
 <xacro:property name="workcell_length" value="8.0"/>
@@ -8,5 +6,5 @@
 <xacro:property name="workcell_thickness" value="0.01"/>
 <xacro:property name="workcell_z" value="-0.1"/>
-<xacro:macro name="ucla_linear_track_demo_cell" params="prefix">
+<xacro:macro name="simple_linear_track_demo_cell" params="prefix">
   <link name="demo_cell_base_link"/>
   <material name="workcell_material">
@@ -101,24 +99,4 @@
     </collision>
   </link>
-  <link name="rail">
-    <visual>
-      <origin xyz="0 0 0"/>
-      <geometry>
-        <box size="4 ${rail_cross_section} ${rail_cross_section}"/>
-      </geometry>
-      <material name="yellow">
-       <color rgba="1.0 1.0 0 1.0"/>
-      </material>
-    </visual>
-    <collision>
-      <origin xyz="0 0 0"/>
-      <geometry>
-        <box size="4 0.1 0.1"/>
-      </geometry>
-      <material name="yellow">
-       <color rgba="1.0 1.0 0 1.0"/>
-      </material>
-    </collision>
-  </link>
   <joint name="cell_base_to_bounds" type="fixed">
     <parent link="demo_cell_base_link" />
@@ -126,16 +104,4 @@
     <origin xyz="0 0 ${workcell_z}"/>
   </joint>
-  <joint name="cell_base_to_rail" type="fixed">
-    <parent link="demo_cell_base_link" />
-    <child link="rail" />
-    <origin xyz="0 0 0"/>
-  </joint>
-  <joint name="rail_to_robot_base_link" type="prismatic">
-    <parent link="rail" />
-    <child link="base_link" />
-    <origin xyz="0 0 ${0.5*rail_cross_section}"/>
-    <axis xyz="1 0 0"/>
-    <limit lower="-2" upper="2" effort="1" velocity="1"/>
-  </joint>
 </xacro:macro>
 </robot>

Commit message: ikfast works with irb2400+linear track.

File: framefab_robot/abb/framefab_irb2400/framefab_irb2400_support/urdf/irb2400_with_linear_track.urdf (robot description, URDF)
Before this commit: robot irb2400_workspace, 10 links, 9 joints
Links:
- added link world_frame
Joints:
- added joint world_to_rail: type fixed, parent world_frame, child rail, origin xyz=0 0 0

File: framefab_robot/abb/framefab_irb2400/framefab_irb2400_support/urdf/irb2400_with_linear_track.xacro (robot description, xacro)
@@ -1,11 +1,18 @@
 <?xml version="1.0" ?>
-<robot name="irb2400_workspace" xmlns:xacro="http://ros.org/wiki/xacro">
+<robot name="framefab_irb2400" xmlns:xacro="http://ros.org/wiki/xacro">
   <!--robot-->
   <xacro:include filename="$(find abb_irb2400_support)/urdf/irb2400_macro.xacro"/>
 	<!--linear track setup-->
 	<xacro:include filename="$(find framefab_irb2400_support)/urdf/simple_linear_track_macro.xacro"/>
+  <link name="world_frame"/>
   <!-- instantiating arm  -->
   <xacro:abb_irb2400 prefix=""/>
 	<!-- linear track  -->
   <xacro:simple_linear_track prefix=""/>
+	<!--bind the rail to word_frame-->
+  <joint name="world_to_rail" type="fixed">
+    <parent link="world_frame" />
+    <child link="rail" />
+    <origin xyz="0 0 0"/>
+  </joint>
 </robot>

File: framefab_robot/abb/framefab_irb2400/framefab_irb2400_support/urdf/irb2400_with_linear_track_workspace.xacro (robot description, xacro)
@@ -1,4 +1,4 @@
 <?xml version="1.0" ?>
-<robot name="irb2400_workspace" xmlns:xacro="http://ros.org/wiki/xacro">
+<robot name="framefab_irb2400" xmlns:xacro="http://ros.org/wiki/xacro">
   <!--robot-->
   <xacro:include filename="$(find abb_irb2400_support)/urdf/irb2400_macro.xacro"/>
@@ -24,8 +24,9 @@
 		<origin xyz="0 0 0" rpy="0 0 0"/>
 	</joint>
-  <joint name="world_to_demo_cell" type="fixed">
-    <parent link="world_frame"/>
-    <child link="demo_cell_base_link"/>
-    <origin xyz="0 0 0" rpy="0 0 0"/>
+	<!--bind the rail to word_frame-->
+  <joint name="world_to_rail" type="fixed">
+    <parent link="world_frame" />
+    <child link="rail" />
+    <origin xyz="0 0 0"/>
   </joint>
 </robot>

File: framefab_robot/abb/framefab_irb2400/framefab_irb2400_support/urdf/simple_linear_track_demo_cell_macro.xacro (robot description, xacro)
@@ -7,5 +7,4 @@
 <xacro:property name="workcell_z" value="-0.1"/>
 <xacro:macro name="simple_linear_track_demo_cell" params="prefix">
-  <link name="demo_cell_base_link"/>
   <material name="workcell_material">
    <color rgba="0.8 1.0 0.8 0.2"/>
@@ -100,5 +99,5 @@
   </link>
   <joint name="cell_base_to_bounds" type="fixed">
-    <parent link="demo_cell_base_link" />
+    <parent link="world_frame" />
     <child link="workcell_bounds" />
     <origin xyz="0 0 ${workcell_z}"/>

File: framefab_robot/abb/framefab_irb2400/framefab_irb2400_support/urdf/simple_linear_track_macro.xacro (robot description, xacro)
@@ -4,5 +4,4 @@
 <xacro:property name="rail_cross_section" value="0.1"/>
 <xacro:macro name="simple_linear_track" params="prefix">
-<!--  <link name="demo_cell_base_link"/>-->
   <link name="rail">
     <visual>
@@ -25,9 +24,4 @@
     </collision>
   </link>
-<!--  <joint name="cell_base_to_rail" type="fixed">-->
-<!--    <parent link="demo_cell_base_link" />-->
-<!--    <child link="rail" />-->
-<!--    <origin xyz="0 0 0"/>-->
-<!--  </joint>-->
   <joint name="rail_to_robot_base_link" type="prismatic">
     <parent link="rail" />
