Commit message: irb2400+track ikfast plugin added.

File: framefab_robot/abb/framefab_irb2400/framefab_irb2400_support/urdf/irb2400_with_linear_track_workspace.urdf (robot description, URDF)
Before this commit: robot framefab_irb2400, 11 links, 10 joints
Links:
- added link eef_frame
- added link hotend_tool; collision mesh filename=package://asw_end_effector/meshes/collision/asw_hotend_end_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 scale=.001 .001 .001; visual mesh filename=package://asw_end_effector/meshes/visual/asw_hotend_end_eff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 scale=.001 .001 .001
- added link tcp_frame
- added link tmp_tcp_frame
- added link workcell_bounds; collision box size=0.01 5.0 3.0; collision box size=0.01 5.0 3.0
Joints:
- added joint cell_base_to_bounds: type fixed, parent world_frame, child workcell_bounds, origin xyz=0 0 -0.1
- added joint eef_frame_to_hotend_tool: type fixed, parent eef_frame, child hotend_tool, origin xyz=0.000088 0.000769 -0.002121 rpy=0 0 0
- added joint eef_to_hotend_tcp_frame: type fixed, parent eef_frame, child tmp_tcp_frame, origin xyz=0.150539 0.001052 0.119157 rpy=0 1.57079632679 0
- added joint link_t_to_eef: type fixed, parent tool0, child eef_frame, origin xyz=0 0 0 rpy=0 0 0
- added joint tmp_to_tcp_frame: type fixed, parent tmp_tcp_frame, child tcp_frame, origin xyz=0 0 0.0

File: framefab_robot/abb/framefab_irb2400/framefab_irb2400_support/urdf/irb2400_with_linear_track_workspace.xacro (robot description, xacro)
@@ -1,4 +1,4 @@
 <?xml version="1.0" ?>
-<robot name="framefab_irb2400" xmlns:xacro="http://ros.org/wiki/xacro">
+<robot name="framefab_irb2400_workspace" xmlns:xacro="http://ros.org/wiki/xacro">
   <!--robot-->
   <xacro:include filename="$(find abb_irb2400_support)/urdf/irb2400_macro.xacro"/>
