Commit message: reformat using A5's robot xacro setup as a template.

File: framefab_robot/abb/framefab_irb2400/framefab_irb2400_support/urdf/irb2400_with_linear_track_workspace.xacro (robot description, xacro)
@@ -1,32 +1,39 @@
 <?xml version="1.0" ?>
 <robot name="framefab_irb2400_workspace" xmlns:xacro="http://ros.org/wiki/xacro">
-  <!--robot-->
+	<xacro:include filename="$(find a5_support)/urdf/resources/materials.xacro"/>
   <xacro:include filename="$(find abb_irb2400_support)/urdf/irb2400_macro.xacro"/>
-	<!--end effector-->
 	<xacro:include filename="$(find asw_end_effector)/urdf/asw_eef_macro.xacro"/>
-	<!--linear track setup-->
-	<xacro:include filename="$(find framefab_irb2400_support)/urdf/simple_linear_track_macro.xacro"/>
-	<!--workcell setup-->
-	<xacro:include filename="$(find framefab_irb2400_support)/urdf/simple_linear_track_demo_cell_macro.xacro"/>
-  <link name="world_frame"/>
-  <!-- instantiating arm  -->
-  <xacro:abb_irb2400 prefix=""/>
-  <!-- instantiating end effector  -->
-  <xacro:asw_eef_definition prefix=""/>
-	<!-- linear track  -->
-  <xacro:simple_linear_track prefix=""/>
-  <!-- workcell  -->
-  <xacro:simple_linear_track_demo_cell prefix=""/>
-	<!-- Attach the end effector to the end of the robot arm (tool0) -->
-	<joint name="link_t_to_eef" type="fixed">
+	<xacro:include filename="$(find ucla_linear_axis)/urdf/ucla_linear_axis_macro.xacro"/>
+	<!--	<xacro:include filename="$(find framefab_irb2400_support)/urdf/simple_linear_track_demo_cell_macro.xacro"/>-->
+  <xacro:abb_irb2400 prefix="robot_"/>
+  <xacro:asw_eef_definition prefix="eef_"/>
+  <xacro:ucla_linear_axis prefix="linear_axis_"/>
+	<!--  <xacro:simple_linear_track_demo_cell prefix=""/>-->
+	<!-- Link list -->
+	<link name="world_frame"/>
+  <link name="base_link"/>
+	<!-- End of link list -->
+	<!-- Joint list -->
+	<!--bind the rail to word_frame, can be disabled if using modile platform-->
+  <joint name="world_to_base_link" type="fixed">
+    <parent link="world_frame" />
+    <child link="base_link" />
+    <origin xyz="0 0 0"/>
+  </joint>
+	<joint name="linear_axis_to_base_link" type="fixed">
+    <origin xyz="0 0 0" rpy="0 0 0"/>
+    <parent link="base_link"/>
+    <child link="linear_axis_base_link"/>
+  </joint>
+  <joint name="robot_to_linear_axis" type="fixed">
+    <origin xyz="0 0 0" rpy="0 0 0"/>
+    <parent link="linear_axis_robot_mount"/>
+    <child link="robot_base_link"/>
+  </joint>
+	<joint name="ee_to_robot" type="fixed">
 		<parent link="tool0"/>
-		<child link="eef_frame"/>
+		<child link="eef_base_link"/>
 		<origin xyz="0 0 0" rpy="0 0 0"/>
 	</joint>
-	<!--bind the rail to word_frame-->
-  <joint name="world_to_rail" type="fixed">
-    <parent link="world_frame" />
-    <child link="rail" />
-    <origin xyz="0 0 0"/>
-  </joint>
+	<!-- End of joint list -->
 </robot>

File: framefab_robot/asw_end_effector/urdf/asw_eef_macro.xacro (robot description, xacro)
@@ -1,46 +1,40 @@
 <?xml version="1.0" ?>
 <robot xmlns:xacro="http://ros.org/wiki/xacro">
-  <xacro:property name="hotend_tcp_x" value="0.150539"/>
-  <xacro:property name="hotend_tcp_y" value="0.001052"/>
-  <xacro:property name="hotend_tcp_z" value="0.119157"/>
-  <xacro:property name="half_pi" value="1.5707963267948966"/>
-  <xacro:macro name="asw_eef_definition" params="prefix">
-    <!-- eef_frame is Base Link -->
-    <link name="${prefix}eef_frame"/>
-    <link name="${prefix}hotend_tool">
-      <visual>
-        <geometry>
-          <mesh filename="package://asw_end_effector/meshes/visual/asw_hotend_end_effector.stl" scale=".001 .001 .001"/>
-        </geometry>
-        <material name="grey">
-          <color rgba="0.5 0.5 0.5 1.0"/>
-        </material>
-      </visual>
-      <collision>
-        <geometry>
-          <mesh filename="package://asw_end_effector/meshes/collision/asw_hotend_end_effector_shrinked_tip-4mm.stl" scale=".001 .001 .001"/>
-        </geometry>
-        <material name="red">
-          <color rgba="1 0 0 1"/>
-        </material>
-      </collision>
-    </link>
-    <joint name="${prefix}eef_frame_to_hotend_tool" type="fixed">
-        <parent link="${prefix}eef_frame"/>
-        <child link="${prefix}hotend_tool"/>
-        <origin xyz="0.000088 0.000769 -0.002121" rpy="0 0 0"/>
-    </joint>
-    <link name="${prefix}tmp_tcp_frame"/> <!--The actual 'useful' work frame-->
-    <link name="${prefix}tcp_frame"/> <!--The actual 'useful' work frame-->
-    <joint name="${prefix}eef_to_hotend_tcp_frame" type="fixed">
-        <parent link="${prefix}eef_frame"/>
-        <child link="${prefix}tmp_tcp_frame"/>
-        <origin xyz="${hotend_tcp_x} ${hotend_tcp_y} ${hotend_tcp_z}" rpy="0 ${half_pi} 0"/>
-    </joint>
-    <joint name="${prefix}tmp_to_tcp_frame" type="fixed">
-        <parent link="${prefix}tmp_tcp_frame"/>
-        <child link="${prefix}tcp_frame"/>
-        <origin xyz="0 0 0.0"/>
-    </joint>
+  <xacro:macro name="asw_eef" params="prefix">
+  <xacro:property name="tcp_cal_filename" value="$(find asw_end_effector)/config/tcp_calibration.yaml"/>
+  <xacro:property name="tcp_cal" value="${load_yaml(tcp_cal_filename)}" />
+  <xacro:property name="eef_mount_offset_filename" value="$(find asw_end_effector)/config/eef_mount_offset.yaml"/>
+  <xacro:property name="eef_mount_offset" value="${load_yaml(eef_mount_offset_filename)}" />
+	<!-- link list -->
+  <link name="${prefix}base_link"/>
+    <visual>
+    	<origin xyz="${eef_mount_offset['transform']['x']} ${eef_mount_offset['transform']['y']} ${eef_mount_offset['transform']['z']}" rpy="0 0 0"/>
+      <geometry>
+        <mesh filename="package://asw_end_effector/meshes/visual/asw_hotend_end_effector.stl" scale=".001 .001 .001"/>
+      </geometry>
+      <material name="grey">
+        <color rgba="0.5 0.5 0.5 1.0"/>
+      </material>
+    </visual>
+    <collision>
+    	<origin xyz="${eef_mount_offset['transform']['x']} ${eef_mount_offset['transform']['y']} ${eef_mount_offset['transform']['z']}" rpy="0 0 0"/>
+      <geometry>
+        <mesh filename="package://asw_end_effector/meshes/collision/asw_hotend_end_effector_shrinked_tip-4mm.stl" scale=".001 .001 .001"/>
+      </geometry>
+      <material name="red">
+        <color rgba="1 0 0 1"/>
+      </material>
+    </collision>
+  </link>
+	<link name="${prefix}tcp_frame"/>
+	<!-- end of link list -->
+	<!-- joint list -->
+  <joint name="${prefix}base_to_tcp" type="fixed">
+		<origin xyz="${tcp_cal['transform']['x']} ${tcp_cal['transform']['y']} ${tcp_cal['transform']['z']}"
+              rpy="${tcp_cal['transform']['roll']} ${tcp_cal['transform']['pitch']} ${tcp_cal['transform']['yaw']}"/>
+    <parent link="${prefix}base_link"/>
+    <child link="${prefix}tcp_frame"/>
+  </joint>
+	<!-- end of joint list -->
   </xacro:macro>
 </robot>

File: framefab_robot/linear_axis/ucla_linear_axis/urdf/ucla_linear_axis_macro.xacro (robot description, xacro)
@@ -3,8 +3,6 @@
 	<xacro:property name="half_pi" value="1.5707963267948966"/>
 	<xacro:macro name="ucla_linear_axis" params="prefix">
-<!--inherent from target robot model-->
-<!--	<link name="${prefix}link_4_mount_point"/>-->
-<!--	<link name="${prefix}material_feeder">-->
-	<link name="${prefix}linear_axis">
+	<!--	Link list-->
+	<link name="${prefix}base_link">
 	  <visual>
 		<geometry>
@@ -24,9 +22,27 @@
 	  </collision>
 	</link>
-<!--	<joint name="${prefix}link_4_mount_point_to_material_feeder" type="fixed">-->
-<!--		<parent link="${prefix}link_4_mount_point"/>-->
-<!--		<child link="${prefix}material_feeder"/>-->
-<!--		<origin xyz="0 0 0" rpy="0 0 0"/>-->
-<!--	</joint>-->
+	<link name="${prefix}zero"/>
+	<link name="${prefix}carriage"/>
+	<link name="${prefix}robot_mount"/>
+	<!--	End of link list-->
+	<!-- Joint list -->
+  <joint name="${prefix}joint_1" type="fixed">
+    <parent link="${prefix}base_link"/>
+    <child link="${prefix}zero"/>
+    <origin xyz="$0.0 0.0 0.0" rpy="0 0 0"/>
+  </joint>
+  <joint name="${prefix}actuation_joint" type="prismatic">
+    <parent link="${prefix}zero"/>
+    <child link="${prefix}carriage"/>
+    <origin xyz="0 0 0" rpy="0 0 0"/>
+    <axis xyz="1 0 0"/>
+    <limit lower="-5.750" upper="-0.010" effort="0" velocity="0.150"/>
+  </joint>
+	<joint name="${prefix}joint_3" type="fixed">
+    <parent link="${prefix}carriage"/>
+    <child link="${prefix}robot_mount"/>
+    <origin xyz="0 0 0" rpy="0 0 0"/>
+  </joint>
+	<!-- End of joint list -->
 	</xacro:macro>
 </robot>
