Commit message: irb2400 + simple track ikfast generation fails. Customized ikfast doc init.

File: framefab_robot/abb/framefab_irb6600/framefab_irb6600_support/urdf/irb2400_with_simple_track_workspace.xacro (robot description, xacro)
@@ -1,13 +1,13 @@
 <?xml version="1.0" ?>
-<robot name="framefab_irb6600_workspace" xmlns:xacro="http://ros.org/wiki/xacro">
+<robot name="framefab_irb2400_simple_track" xmlns:xacro="http://ros.org/wiki/xacro">
 	<xacro:property name="half_pi" value="1.5707963267948966"/>
 	<xacro:include filename="$(find framefab_irb6600_support)/urdf/resources/materials.xacro"/>
-  <xacro:include filename="$(find abb_irb6600_support)/urdf/irb6640_macro.xacro"/>
+  <xacro:include filename="$(find abb_irb2400_support)/urdf/irb2400_macro.xacro"/>
 	<xacro:include filename="$(find asw_end_effector)/urdf/asw_eef_macro.xacro"/>
-	<xacro:include filename="$(find ucla_linear_axis)/urdf/ucla_linear_axis_macro.xacro"/>
+	<xacro:include filename="$(find framefab_irb6600_support)/urdf/simple_linear_track_macro.xacro"/>
 	<!--	<xacro:include filename="$(find framefab_irb6600_support)/urdf/simple_linear_track_demo_cell_macro.xacro"/>-->
-  <xacro:abb_irb6640 prefix="robot_"/>
+  <xacro:abb_irb2400 prefix="robot_"/>
   <xacro:asw_eef prefix="eef_"/>
-  <xacro:ucla_linear_axis prefix="linear_axis_"/>
+  <xacro:simple_linear_track prefix="linear_axis_"/>
 	<!--  <xacro:simple_linear_track_demo_cell prefix=""/>-->
 	<!-- Link list -->

File: framefab_robot/abb/framefab_irb6600/framefab_irb6600_support/urdf/irb6600_with_linear_track_workspace.urdf (robot description, URDF)
Before this commit: robot framefab_irb6600_workspace, 19 links, 18 joints
Links:
- removed link world_frame
Joints:
- removed joint world_to_base_link

File: framefab_robot/abb/framefab_irb6600/framefab_irb6600_support/urdf/simple_linear_track_macro.xacro (robot description, xacro)
@@ -4,7 +4,7 @@
 <xacro:property name="rail_cross_section" value="0.1"/>
 <xacro:macro name="simple_linear_track" params="prefix">
-  <link name="rail">
+	<!--	Link list-->
+  <link name="${prefix}base_link">
     <visual>
-      <origin xyz="0 0 0"/>
       <geometry>
         <box size="4 ${rail_cross_section} ${rail_cross_section}"/>
@@ -24,11 +24,15 @@
     </collision>
   </link>
-  <joint name="rail_to_robot_base_link" type="prismatic">
-    <parent link="rail" />
-    <child link="base_link" />
+	<link name="${prefix}robot_mount"/>
+	<!--	End of link list-->
+	<!-- Joint list -->
+  <joint name="${prefix}actuation_joint" type="prismatic">
+    <parent link="${prefix}base_link" />
+    <child link="${prefix}robot_mount" />
     <origin xyz="0 0 ${0.5*rail_cross_section}"/>
     <axis xyz="1 0 0"/>
     <limit lower="-2" upper="2" effort="1" velocity="1"/>
   </joint>
+	<!-- End of joint list -->
 </xacro:macro>
 </robot>
