Commit message: ikfast generation failed on simple 6dof case. I have doubt on the sympy version on lab's computer.

File: framefab_robot/abb/framefab_irb6600/framefab_irb6600_support/urdf/irb2400_with_simple_track_workspace.urdf (robot description, URDF)
Before this commit: robot framefab_irb2400_simple_track, 14 links, 13 joints
Links:
- removed link eef_base_link
- removed link eef_tcp_frame
- removed link linear_axis_base_link
- removed link linear_axis_robot_mount
Joints:
- removed joint ee_to_robot
- removed joint eef_base_to_tcp
- removed joint linear_axis_actuation_joint
- removed joint linear_axis_to_base_link
- removed joint robot_to_linear_axis
- added joint robot_to_base_link: type fixed, parent base_link, child robot_base_link, origin xyz=0 0 0 rpy=0 0 0

File: framefab_robot/abb/framefab_irb6600/framefab_irb6600_support/urdf/irb2400_with_simple_track_workspace.xacro (robot description, xacro)
@@ -4,10 +4,10 @@
 	<xacro:include filename="$(find framefab_irb6600_support)/urdf/resources/materials.xacro"/>
   <xacro:include filename="$(find abb_irb2400_support)/urdf/irb2400_macro.xacro"/>
-	<xacro:include filename="$(find asw_end_effector)/urdf/asw_eef_macro.xacro"/>
-	<xacro:include filename="$(find framefab_irb6600_support)/urdf/simple_linear_track_macro.xacro"/>
+<!--	<xacro:include filename="$(find framefab_irb6600_support)/urdf/simple_linear_track_macro.xacro"/>-->
+	<!--	<xacro:include filename="$(find asw_end_effector)/urdf/asw_eef_macro.xacro"/>-->
 	<!--	<xacro:include filename="$(find framefab_irb6600_support)/urdf/simple_linear_track_demo_cell_macro.xacro"/>-->
   <xacro:abb_irb2400 prefix="robot_"/>
-  <xacro:asw_eef prefix="eef_"/>
-  <xacro:simple_linear_track prefix="linear_axis_"/>
+<!--  <xacro:asw_eef prefix="eef_"/>-->
+<!--  <xacro:simple_linear_track prefix="linear_axis_"/>-->
 	<!--  <xacro:simple_linear_track_demo_cell prefix=""/>-->
 	<!-- Link list -->
@@ -15,20 +15,25 @@
 	<!-- End of link list -->
 	<!-- Joint list -->
-	<!--bind the rail to word_frame, can be disabled if using modile platform-->
-	<joint name="linear_axis_to_base_link" type="fixed">
-    <origin xyz="0 0 0" rpy="0 0 ${half_pi}"/>
+	<joint name="robot_to_base_link" type="fixed">
+    <origin xyz="0 0 0" rpy="0 0 0"/>
     <parent link="base_link"/>
-    <child link="linear_axis_base_link"/>
-  </joint>
-  <joint name="robot_to_linear_axis" type="fixed">
-    <origin xyz="0 0 0" rpy="0 0 -${half_pi}"/>
-    <parent link="linear_axis_robot_mount"/>
     <child link="robot_base_link"/>
   </joint>
-	<joint name="ee_to_robot" type="fixed">
-		<parent link="robot_tool0"/>
-		<child link="eef_base_link"/>
-		<origin xyz="0 0 0" rpy="0 0 0"/>
-	</joint>
+	<!--bind the rail to word_frame, can be disabled if using modile platform-->
+<!--	<joint name="linear_axis_to_base_link" type="fixed">-->
+<!--    <origin xyz="0 0 0" rpy="0 0 ${half_pi}"/>-->
+<!--    <parent link="base_link"/>-->
+<!--    <child link="linear_axis_base_link"/>-->
+<!--  </joint>-->
+<!--  <joint name="robot_to_linear_axis" type="fixed">-->
+<!--    <origin xyz="0 0 0" rpy="0 0 -${half_pi}"/>-->
+<!--    <parent link="linear_axis_robot_mount"/>-->
+<!--    <child link="robot_base_link"/>-->
+<!--  </joint>-->
+<!--	<joint name="ee_to_robot" type="fixed">-->
+<!--		<parent link="robot_tool0"/>-->
+<!--		<child link="eef_base_link"/>-->
+<!--		<origin xyz="0 0 0" rpy="0 0 0"/>-->
+<!--	</joint>-->
 	<!-- End of joint list -->
 </robot>

Commit message: add ikfast config references to the doc.

File: framefab_robot/abb/framefab_irb6600/framefab_irb6600_support/urdf/irb2400_with_simple_track_workspace.urdf (robot description, URDF)
Before this commit: robot framefab_irb2400_simple_track, 10 links, 9 joints
Joints:
- joint robot_to_base_link: origin xyz=0 0 0 rpy=0 0 0 -> xyz=0 0 0 rpy=0 0 1.57079632679

File: framefab_robot/abb/framefab_irb6600/framefab_irb6600_support/urdf/irb2400_with_simple_track_workspace.xacro (robot description, xacro)
@@ -16,5 +16,5 @@
 	<!-- Joint list -->
 	<joint name="robot_to_base_link" type="fixed">
-    <origin xyz="0 0 0" rpy="0 0 0"/>
+    <origin xyz="0 0 0" rpy="0 0 ${half_pi}"/>
     <parent link="base_link"/>
     <child link="robot_base_link"/>

Commit message: add some sh scripts to automate the xacro to ikfast workflow a bit.

File: framefab_robot/abb/framefab_irb6600/framefab_irb6600_support/urdf/irb2400_with_simple_track_workspace.urdf (robot description, URDF)
Before this commit: robot framefab_irb2400_simple_track, 10 links, 9 joints
Links:
- added link linear_axis_base_link; collision box size=4 0.1 0.1; visual box size=4 0.1 0.1
Joints:
- removed joint robot_to_base_link
- added joint actuation_joint: type prismatic, parent linear_axis_base_link, child robot_base_link, origin xyz=0 0 0.05, axis 1 0 0, limit lower=-2 upper=2 effort=1 velocity=0.1
- added joint linear_axis_to_base_link: type fixed, parent base_link, child linear_axis_base_link, origin xyz=0 0 0 rpy=0 0 1.57079632679

File: framefab_robot/abb/framefab_irb6600/framefab_irb6600_support/urdf/irb2400_with_simple_track_workspace.xacro (robot description, xacro)
@@ -4,10 +4,10 @@
 	<xacro:include filename="$(find framefab_irb6600_support)/urdf/resources/materials.xacro"/>
   <xacro:include filename="$(find abb_irb2400_support)/urdf/irb2400_macro.xacro"/>
-<!--	<xacro:include filename="$(find framefab_irb6600_support)/urdf/simple_linear_track_macro.xacro"/>-->
+	<xacro:include filename="$(find framefab_irb6600_support)/urdf/simple_linear_track_macro.xacro"/>
 	<!--	<xacro:include filename="$(find asw_end_effector)/urdf/asw_eef_macro.xacro"/>-->
 	<!--	<xacro:include filename="$(find framefab_irb6600_support)/urdf/simple_linear_track_demo_cell_macro.xacro"/>-->
   <xacro:abb_irb2400 prefix="robot_"/>
 <!--  <xacro:asw_eef prefix="eef_"/>-->
-<!--  <xacro:simple_linear_track prefix="linear_axis_"/>-->
+  <xacro:simple_linear_track prefix="linear_axis_"/>
 	<!--  <xacro:simple_linear_track_demo_cell prefix=""/>-->
 	<!-- Link list -->
@@ -15,15 +15,15 @@
 	<!-- End of link list -->
 	<!-- Joint list -->
-	<joint name="robot_to_base_link" type="fixed">
+<!--	<joint name="robot_to_base_link" type="fixed">-->
+<!--    <origin xyz="0 0 0" rpy="0 0 ${half_pi}"/>-->
+<!--    <parent link="base_link"/>-->
+<!--    <child link="robot_base_link"/>-->
+<!--  </joint>-->
+<!--	bind the rail to word_frame, can be disabled if using modile platform-->
+	<joint name="linear_axis_to_base_link" type="fixed">
     <origin xyz="0 0 0" rpy="0 0 ${half_pi}"/>
     <parent link="base_link"/>
-    <child link="robot_base_link"/>
+    <child link="linear_axis_base_link"/>
   </joint>
-	<!--bind the rail to word_frame, can be disabled if using modile platform-->
-<!--	<joint name="linear_axis_to_base_link" type="fixed">-->
-<!--    <origin xyz="0 0 0" rpy="0 0 ${half_pi}"/>-->
-<!--    <parent link="base_link"/>-->
-<!--    <child link="linear_axis_base_link"/>-->
-<!--  </joint>-->
 <!--  <joint name="robot_to_linear_axis" type="fixed">-->
 <!--    <origin xyz="0 0 0" rpy="0 0 -${half_pi}"/>-->
@@ -31,4 +31,11 @@
 <!--    <child link="robot_base_link"/>-->
 <!--  </joint>-->
+  <joint name="actuation_joint" type="prismatic">
+    <parent link="linear_axis_base_link" />
+    <child link="robot_base_link" />
+    <origin xyz="0 0 0.05"/>
+    <axis xyz="1 0 0"/>
+    <limit lower="-2" upper="2" effort="1" velocity="0.1"/>
+  </joint>
 <!--	<joint name="ee_to_robot" type="fixed">-->
 <!--		<parent link="robot_tool0"/>-->

File: framefab_robot/abb/framefab_irb6600/framefab_irb6600_support/urdf/simple_linear_track_macro.xacro (robot description, xacro)
@@ -7,4 +7,5 @@
   <link name="${prefix}base_link">
     <visual>
+      <origin xyz="0 0 0"/>
       <geometry>
         <box size="4 ${rail_cross_section} ${rail_cross_section}"/>
@@ -17,5 +18,5 @@
       <origin xyz="0 0 0"/>
       <geometry>
-        <box size="4 0.1 0.1"/>
+        <box size="4 ${rail_cross_section} ${rail_cross_section}"/>
       </geometry>
       <material name="yellow">
@@ -24,14 +25,14 @@
     </collision>
   </link>
-	<link name="${prefix}robot_mount"/>
+<!--	<link name="${prefix}robot_mount"/>-->
 	<!--	End of link list-->
 	<!-- Joint list -->
-  <joint name="${prefix}actuation_joint" type="prismatic">
-    <parent link="${prefix}base_link" />
-    <child link="${prefix}robot_mount" />
-    <origin xyz="0 0 ${0.5*rail_cross_section}"/>
-    <axis xyz="1 0 0"/>
-    <limit lower="-2" upper="2" effort="1" velocity="1"/>
-  </joint>
+<!--  <joint name="${prefix}actuation_joint" type="prismatic">-->
+<!--    <parent link="${prefix}base_link" />-->
+<!--    <child link="${prefix}robot_mount" />-->
+<!--    <origin xyz="0 0 ${0.5*rail_cross_section}"/>-->
+<!--    <axis xyz="1 0 0"/>-->
+<!--    <limit lower="-2" upper="2" effort="1" velocity="0.1"/>-->
+<!--  </joint>-->
 	<!-- End of joint list -->
 </xacro:macro>

Commit message: add more info to ikfast tutorial.

File: framefab_robot/abb/framefab_irb6600/framefab_irb6600_support/urdf/irb2400_with_simple_track_workspace.urdf (robot description, URDF)
Before this commit: robot framefab_irb2400_simple_track, 11 links, 10 joints
Joints:
- joint linear_axis_to_base_link: origin xyz=0 0 0 rpy=0 0 1.57079632679 -> xyz=0 0 0 rpy=0 0 0

File: framefab_robot/abb/framefab_irb6600/framefab_irb6600_support/urdf/irb2400_with_simple_track_workspace.xacro (robot description, xacro)
@@ -22,5 +22,5 @@
 <!--	bind the rail to word_frame, can be disabled if using modile platform-->
 	<joint name="linear_axis_to_base_link" type="fixed">
-    <origin xyz="0 0 0" rpy="0 0 ${half_pi}"/>
+    <origin xyz="0 0 0" rpy="0 0 0"/>
     <parent link="base_link"/>
     <child link="linear_axis_base_link"/>
