Commit message: abb execution working: need to enable robot_state in rviz (not the one in movegroup), speed up traj and diable linear track's speed limit.

File: framefab_robot/abb/framefab_irb6600/framefab_irb6600_support/urdf/irb6600_with_linear_track_workspace.urdf (robot description, URDF)
Before this commit: robot framefab_irb6600_workspace, 18 links, 17 joints
Joints:
- joint linear_axis_actuation_joint: limit lower=0 upper=5.4 effort=0 velocity=0.150 -> lower=0 upper=5.4 effort=1 velocity=1

File: framefab_robot/asw_end_effector/urdf/asw_eef_macro.xacro (robot description, xacro)
@@ -1,4 +1,3 @@
 <?xml version="1.0" ?>
-<<<<<<< HEAD
 <robot xmlns:xacro="http://ros.org/wiki/xacro">
   <xacro:macro name="asw_eef" params="prefix">
@@ -39,49 +38,3 @@
 		<!-- end of joint list -->
 	</xacro:macro>
-=======
-<robot xmlns:xacro="http://wiki.ros.org/xacro">
-  <xacro:property name="hotend_tcp_x" value="0.150539"/>
-  <xacro:property name="hotend_tcp_y" value="0.001052"/>
-  <xacro:property name="hotend_tcp_z" value="0.119157"/>
-  <xacro:property name="half_pi" value="1.5707963267948966"/>
-  <xacro:macro name="asw_eef_definition" params="prefix">
-    <!-- eef_frame is Base Link -->
-    <link name="${prefix}eef_frame"/>
-    <link name="${prefix}hotend_tool">
-      <visual>
-        <geometry>
-          <mesh filename="package://asw_end_effector/meshes/visual/asw_hotend_end_effector.stl" scale=".001 .001 .001"/>
-        </geometry>
-        <material name="grey">
-          <color rgba="0.5 0.5 0.5 1.0"/>
-        </material>
-      </visual>
-      <collision>
-        <geometry>
-          <mesh filename="package://asw_end_effector/meshes/collision/asw_hotend_end_effector_shrinked_tip-4mm.stl" scale=".001 .001 .001"/>
-        </geometry>
-        <material name="red">
-          <color rgba="1 0 0 1"/>
-        </material>
-      </collision>
-    </link>
-    <joint name="${prefix}eef_frame_to_hotend_tool" type="fixed">
-        <parent link="${prefix}eef_frame"/>
-        <child link="${prefix}hotend_tool"/>
-        <origin xyz="0.000088 0.000769 -0.002121" rpy="0 0 0"/>
-    </joint>
-    <link name="${prefix}tmp_tcp_frame"/> <!--The actual 'useful' work frame-->
-    <link name="${prefix}tcp_frame"/> <!--The actual 'useful' work frame-->
-    <joint name="${prefix}eef_to_hotend_tcp_frame" type="fixed">
-        <parent link="${prefix}eef_frame"/>
-        <child link="${prefix}tmp_tcp_frame"/>
-        <origin xyz="${hotend_tcp_x} ${hotend_tcp_y} ${hotend_tcp_z}" rpy="0 ${half_pi} 0"/>
-    </joint>
-    <joint name="${prefix}tmp_to_tcp_frame" type="fixed">
-        <parent link="${prefix}tmp_tcp_frame"/>
-        <child link="${prefix}tcp_frame"/>
-        <origin xyz="0 0 0.0"/>
-    </joint>
-  </xacro:macro>
->>>>>>> 31df9306da2bdd7d969b7d837ecf2cfb19e2fbd8
 </robot>

File: framefab_robot/linear_axis/ucla_linear_axis/urdf/ucla_linear_axis_macro.xacro (robot description, xacro)
@@ -47,5 +47,5 @@
     <origin xyz="0 0 0" rpy="0 0 0"/>
     <axis xyz="1 0 0"/>
-    <limit lower="0" upper="5.4" effort="0" velocity="0.150"/>
+    <limit lower="0" upper="5.4" effort="1" velocity="1"/>
   </joint>
 	<joint name="${prefix}joint_3" type="fixed">
