Commit message: finer visual model of material feeder added.

File: framefab_robot/asw_material_feeder/urdf/asw_material_feeder_macro.xacro (robot description, xacro)
@@ -8,5 +8,5 @@
 	  <visual>
 		<geometry>
-		  <mesh filename="package://asw_material_feeder/meshes/visual/asw_material_feeder_collision_model.stl" scale=".001 .001 .001"/>
+		  <mesh filename="package://asw_material_feeder/meshes/visual/asw_material_feeder_visual_model.stl" scale=".001 .001 .001"/>
 		</geometry>
 		<material name="grey">

Commit message: fix #68. Material feeder attached to link 3.

File: framefab_robot/asw_material_feeder/urdf/asw_material_feeder_macro.xacro (robot description, xacro)
@@ -4,5 +4,5 @@
 	<xacro:macro name="asw_material_feeder_definition" params="prefix">
 	<!-- material_feeder_mount_point is Base Link, inherit from host robot -->
-	<link name="${prefix}link_4_mount_point"/>
+	<link name="${prefix}link_3_mount_point"/>
 	<link name="${prefix}material_feeder">
 	  <visual>
@@ -23,6 +23,6 @@
 	  </collision>
 	</link>
-	<joint name="${prefix}link_4_mount_point_to_material_feeder" type="fixed">
-		<parent link="${prefix}link_4_mount_point"/>
+	<joint name="${prefix}link_3_mount_point_to_material_feeder" type="fixed">
+		<parent link="${prefix}link_3_mount_point"/>
 		<child link="${prefix}material_feeder"/>
 		<origin xyz="0 0 0" rpy="0 0 0"/>

File: framefab_robot/kuka/framefab_kr6_r900/framefab_kr6_r900_support/urdf/kr6_r900_workspace.xacro (robot description, xacro)
@@ -5,7 +5,7 @@
 	<xacro:include filename="$(find asw_material_feeder)/urdf/asw_material_feeder_macro.xacro"/>
 	<xacro:include filename="$(find framefab_kr6_r900_support)/urdf/mit_3-412_workspace_micro.xacro"/>
-	<xacro:property name="link4_mount_base_x" value="0.06762"/>
-	<xacro:property name="link4_mount_base_y" value="0.0"/>
-	<xacro:property name="link4_mount_base_z" value="0.0575"/>
+	<xacro:property name="link3_mount_base_x" value="0.06762"/>
+	<xacro:property name="link3_mount_base_y" value="0.0"/>
+	<xacro:property name="link3_mount_base_z" value="0.0925"/>
 	<link name="world_frame"/>
 	<!-- instantiating arm  -->
@@ -23,8 +23,8 @@
 	</joint>
 	<!-- Attach the material feeder to the link4 mount point of the robot arm -->
-    <joint name="link_4_to_link_4_mount_point" type="fixed">
-        <parent link="link_4"/>
-        <child link="link_4_mount_point"/>
-        <origin xyz="${link4_mount_base_x} ${link4_mount_base_y} ${link4_mount_base_z}" rpy="0 0 0"/>
+    <joint name="link_3_to_link_3_mount_point" type="fixed">
+        <parent link="link_3"/>
+        <child link="link_3_mount_point"/>
+        <origin xyz="${link3_mount_base_x} ${link3_mount_base_y} ${link3_mount_base_z}" rpy="0 0 0"/>
     </joint>
 	<!-- start of arm-workcell joint definitions -->

Commit message: new kuka moveit pkg + ikfast plugin generated.

File: framefab_robot/asw_material_feeder/urdf/asw_material_feeder_macro.xacro (robot description, xacro)
@@ -4,5 +4,5 @@
 	<xacro:macro name="asw_material_feeder_definition" params="prefix">
 	<!-- material_feeder_mount_point is Base Link, inherit from host robot -->
-	<link name="${prefix}link_3_mount_point"/>
+	<link name="${prefix}mount_point"/>
 	<link name="${prefix}material_feeder">
 	  <visual>
@@ -23,6 +23,6 @@
 	  </collision>
 	</link>
-	<joint name="${prefix}link_3_mount_point_to_material_feeder" type="fixed">
-		<parent link="${prefix}link_3_mount_point"/>
+	<joint name="mount_point_to_material_feeder" type="fixed">
+		<parent link="${prefix}mount_point"/>
 		<child link="${prefix}material_feeder"/>
 		<origin xyz="0 0 0" rpy="0 0 0"/>

File: framefab_robot/kuka/framefab_kr6_r900/framefab_kr6_r900_support/urdf/kr6_r900_workspace.xacro (robot description, xacro)
@@ -1,39 +1,40 @@
 <?xml version="1.0" ?>
 <robot name="kr6_r900_workspace" xmlns:xacro="http://wiki.ros.org/xacro">
+	<xacro:property name="link3_mount_base_x" value="0.06762"/>
+	<xacro:property name="link3_mount_base_y" value="0.0"/>
+	<xacro:property name="link3_mount_base_z" value="0.0925"/>
  	<xacro:include filename="$(find kuka_kr6_support)/urdf/kr6r900sixx_macro.xacro"/>
 	<xacro:include filename="$(find asw_end_effector)/urdf/asw_eef_macro.xacro"/>
 	<xacro:include filename="$(find asw_material_feeder)/urdf/asw_material_feeder_macro.xacro"/>
 	<xacro:include filename="$(find framefab_kr6_r900_support)/urdf/mit_3-412_workspace_micro.xacro"/>
-	<xacro:property name="link3_mount_base_x" value="0.06762"/>
-	<xacro:property name="link3_mount_base_y" value="0.0"/>
-	<xacro:property name="link3_mount_base_z" value="0.0925"/>
-	<link name="world_frame"/>
 	<!-- instantiating arm  -->
-	<xacro:kuka_kr6r900sixx prefix=""/>
+	<xacro:kuka_kr6r900sixx prefix="robot_"/>
 	<!-- instantiating end effector  -->
-	<xacro:asw_eef_definition prefix=""/>
+	<xacro:asw_eef prefix="eef_"/>
 	<!-- instantiating material feeder  -->
-	<xacro:asw_material_feeder_definition prefix=""/>
-	<xacro:mit_workspace prefix=""/>
+	<xacro:asw_material_feeder_definition prefix="material_feeder_"/>
+	<!-- instantiating workspace  -->
+	<xacro:mit_workspace prefix="workspace_"/>
+	<link name="base_link"/>
 	<!-- Attach the end effector to the end of the robot arm (tool0) -->
-	<joint name="link_t_to_eef" type="fixed">
-		<parent link="tool0"/>
-		<child link="eef_frame"/>
+	<joint name="ee_to_robot" type="fixed">
+		<parent link="robot_tool0"/>
+		<child link="eef_base_link"/>
 		<origin xyz="0 0 0" rpy="0 0 0"/>
 	</joint>
 	<!-- Attach the material feeder to the link4 mount point of the robot arm -->
-    <joint name="link_3_to_link_3_mount_point" type="fixed">
-        <parent link="link_3"/>
-        <child link="link_3_mount_point"/>
-        <origin xyz="${link3_mount_base_x} ${link3_mount_base_y} ${link3_mount_base_z}" rpy="0 0 0"/>
-    </joint>
+  <joint name="link_3_to_link_3_mount_point" type="fixed">
+      <parent link="robot_link_3"/>
+      <child link="material_feeder_mount_point"/>
+      <origin xyz="${link3_mount_base_x} ${link3_mount_base_y} ${link3_mount_base_z}" rpy="0 0 0"/>
+  </joint>
 	<!-- start of arm-workcell joint definitions -->
 	<joint name="world_to_base" type="fixed">
-		<parent link="world_frame"/>
-		<child link="base_link"/>
+		<parent link="base_link"/>
+		<child link="robot_base_link"/>
 		<origin xyz="0 0 0" rpy="0 0 0"/>
 	</joint>
 	<joint name="world_to_workspace" type="fixed">
-		<parent link="world_frame"/>
+		<parent link="base_link"/>
 		<child link="workspace_base_link"/>
 		<origin xyz="0 0 0" rpy="0 0 0"/>

File: framefab_robot/kuka/framefab_kr6_r900/framefab_kr6_r900_support/urdf/mit_3-412_workspace_micro.xacro (robot description, xacro)
@@ -5,6 +5,6 @@
 <robot xmlns:xacro="http://wiki.ros.org/xacro">
 <xacro:macro name="mit_workspace" params="prefix">
-<link name="${prefix}workspace_base_link"/>
-<link name="${prefix}workspace_objects">
+<link name="${prefix}base_link"/>
+<link name="${prefix}objects">
 <visual>
 	<geometry>
@@ -21,7 +21,7 @@
 </collision>
 </link>
-<joint name="${prefix}workspace_baselink_to_objects" type="fixed">
-	<parent link="${prefix}workspace_base_link"/>
-	<child link="${prefix}workspace_objects"/>
+<joint name="${prefix}baselink_to_objects" type="fixed">
+	<parent link="${prefix}base_link"/>
+	<child link="${prefix}objects"/>
 	<origin xyz="0 0 0" rpy="0 0 0"/>
 </joint>
