Commit message: tool frame tf align model.

File: framefab_robot/asw_end_effector/urdf/asw_eef_macro.xacro (robot description, xacro)
@@ -1,7 +1,7 @@
 <?xml version="1.0" ?>
 <robot xmlns:xacro="http://ros.org/wiki/xacro">
-  <xacro:property name="hotend_tcp_x" value="0.15098"/>
-  <xacro:property name="hotend_tcp_y" value="0.000655"/>
-  <xacro:property name="hotend_tcp_z" value="0.115553"/>
+  <xacro:property name="hotend_tcp_x" value="0.15045"/>
+  <xacro:property name="hotend_tcp_y" value="0.000283"/>
+  <xacro:property name="hotend_tcp_z" value="0.121277"/>
   <xacro:property name="half_pi" value="1.5707963267948966"/>
   <xacro:macro name="asw_eef_definition" params="prefix">

File: framefab_robot/kuka/framefab_kr6_r900/framefab_kr6_r900_support/urdf/kr6_r900_workspace.urdf (robot description, URDF)
Before this commit: robot kr6_r900_workspace, 13 links, 12 joints
Joints:
- joint eef_to_hotend_tcp_frame: origin xyz=0.15098 0.000655 0.115553 rpy=0 1.57079632679 0 -> xyz=0.15045 0.000282 0.121277 rpy=0 1.57079632679 0

Commit message: Messing around

File: framefab_robot/asw_end_effector/urdf/asw_eef_macro.xacro (robot description, xacro)
@@ -31,9 +31,15 @@
         <origin xyz="0 0 0" rpy="0 0 0"/>
     </joint>
+    <link name="${prefix}tmp_tcp_frame"/> <!--The actual 'useful' work frame-->
     <link name="${prefix}tcp_frame"/> <!--The actual 'useful' work frame-->
     <joint name="${prefix}eef_to_hotend_tcp_frame" type="fixed">
         <parent link="${prefix}eef_frame"/>
+        <child link="${prefix}tmp_tcp_frame"/>
+        <origin xyz="${hotend_tcp_x} ${hotend_tcp_y} ${hotend_tcp_z}" rpy="0 ${half_pi} 0"/>
+    </joint>
+    <joint name="${prefix}tmp_to_tcp_frame" type="fixed">
+        <parent link="${prefix}tmp_tcp_frame"/>
         <child link="${prefix}tcp_frame"/>
-        <origin xyz="${hotend_tcp_x} ${hotend_tcp_y} ${hotend_tcp_z}" rpy="0 ${half_pi} 0"/>
+        <origin xyz="0 0 0.002"/>
     </joint>
   </xacro:macro>

Commit message: fine-grained eef collision model added. tmp_frame shift changed to 0.

File: framefab_robot/asw_end_effector/urdf/asw_eef_macro.xacro (robot description, xacro)
@@ -19,5 +19,5 @@
       <collision>
         <geometry>
-          <mesh filename="package://asw_end_effector/meshes/collision/asw_hotend_end_effector_hull.stl" scale=".001 .001 .001"/>
+          <mesh filename="package://asw_end_effector/meshes/collision/asw_hotend_end_effector_hull_fine_grained.stl" scale=".001 .001 .001"/>
         </geometry>
         <material name="red">
@@ -41,5 +41,5 @@
         <parent link="${prefix}tmp_tcp_frame"/>
         <child link="${prefix}tcp_frame"/>
-        <origin xyz="0 0 0.002"/>
+        <origin xyz="0 0 0.0"/>
     </joint>
   </xacro:macro>

File: framefab_robot/kuka/framefab_kr6_r900/framefab_kr6_r900_support/urdf/kr6_r900_workspace.xacro (robot description, xacro)
@@ -3,5 +3,5 @@
   <xacro:include filename="$(find kuka_kr6_support)/urdf/kr6r900sixx_macro.xacro"/>
   <xacro:include filename="$(find asw_end_effector)/urdf/asw_eef_macro.xacro"/>
-<!--	<xacro:include filename="$(find framefab_kr6_r900_support)/urdf/mit_3-412_workspace_micro.xacro"/>-->
+	<xacro:include filename="$(find framefab_kr6_r900_support)/urdf/mit_3-412_workspace_micro.xacro"/>
   <link name="world_frame"/>
   <!-- instantiating arm  -->
@@ -9,5 +9,5 @@
   <!-- instantiating end effector  -->
   <xacro:asw_eef_definition prefix=""/>
-<!--	<xacro:mit_workspace prefix=""/>-->
+	<xacro:mit_workspace prefix=""/>
   <!-- Attach the end effector to the end of the robot arm (tool0) -->
   <joint name="link_t_to_eef" type="fixed">
@@ -22,8 +22,8 @@
     <origin xyz="0 0 0" rpy="0 0 0"/>
   </joint>
-<!--  <joint name="world_to_workspace" type="fixed">-->
-<!--    <parent link="world_frame"/>-->
-<!--    <child link="workspace_base_link"/>-->
-<!--    <origin xyz="0 0 0" rpy="0 0 0"/>-->
-<!--  </joint>-->
+  <joint name="world_to_workspace" type="fixed">
+    <parent link="world_frame"/>
+    <child link="workspace_base_link"/>
+    <origin xyz="0 0 0" rpy="0 0 0"/>
+  </joint>
 </robot>

Commit message: update end effector caliberated data and shorten the retraction distance.

File: framefab_robot/asw_end_effector/urdf/asw_eef_macro.xacro (robot description, xacro)
@@ -1,7 +1,7 @@
 <?xml version="1.0" ?>
 <robot xmlns:xacro="http://ros.org/wiki/xacro">
-  <xacro:property name="hotend_tcp_x" value="0.15045"/>
-  <xacro:property name="hotend_tcp_y" value="0.000283"/>
-  <xacro:property name="hotend_tcp_z" value="0.121277"/>
+  <xacro:property name="hotend_tcp_x" value="0.150539"/>
+  <xacro:property name="hotend_tcp_y" value="0.001052"/>
+  <xacro:property name="hotend_tcp_z" value="0.119157"/>
   <xacro:property name="half_pi" value="1.5707963267948966"/>
   <xacro:macro name="asw_eef_definition" params="prefix">

Commit message: CLT initial solution working. Optimality of the solution is indeed important, so let's get into RRT*!

File: framefab_robot/asw_end_effector/urdf/asw_eef_macro.xacro (robot description, xacro)
@@ -29,5 +29,5 @@
         <parent link="${prefix}eef_frame"/>
         <child link="${prefix}hotend_tool"/>
-        <origin xyz="0 0 0" rpy="0 0 0"/>
+        <origin xyz="0.000088 0.000769 -0.002121" rpy="0 0 0"/>
     </joint>
     <link name="${prefix}tmp_tcp_frame"/> <!--The actual 'useful' work frame-->

Commit message: fix #75.

File: framefab_robot/asw_end_effector/urdf/asw_eef_macro.xacro (robot description, xacro)
@@ -19,5 +19,5 @@
       <collision>
         <geometry>
-          <mesh filename="package://asw_end_effector/meshes/collision/asw_hotend_end_effector_hull_fine_grained.stl" scale=".001 .001 .001"/>
+          <mesh filename="package://asw_end_effector/meshes/collision/asw_hotend_end_effector_shrinked_tip-4mm.stl" scale=".001 .001 .001"/>
         </geometry>
         <material name="red">

Commit message: quick fix on retration planning.

File: framefab_robot/asw_end_effector/urdf/asw_eef_macro.xacro (robot description, xacro)
@@ -19,5 +19,5 @@
       <collision>
         <geometry>
-          <mesh filename="package://asw_end_effector/meshes/collision/asw_hotend_end_effector_shrinked_tip-4mm.stl" scale=".001 .001 .001"/>
+          <mesh filename="package://asw_end_effector/meshes/collision/asw_hotend_end_effector_shrinked_tip-12mm.stl" scale=".001 .001 .001"/>
         </geometry>
         <material name="red">

Commit message: hotfix for partial shrinked geometry, refer #69. Minor change in UI (fetched_plan now in increasing order!)

File: framefab_robot/asw_end_effector/urdf/asw_eef_macro.xacro (robot description, xacro)
@@ -19,5 +19,5 @@
       <collision>
         <geometry>
-          <mesh filename="package://asw_end_effector/meshes/collision/asw_hotend_end_effector_shrinked_tip-12mm.stl" scale=".001 .001 .001"/>
+          <mesh filename="package://asw_end_effector/meshes/collision/asw_hotend_end_effector_shrinked_tip-4mm.stl" scale=".001 .001 .001"/>
         </geometry>
         <material name="red">

Commit message: irb6600 + linear axis urdf added.

File: framefab_robot/asw_end_effector/urdf/asw_eef_macro.xacro (robot description, xacro)
@@ -2,39 +2,39 @@
 <robot xmlns:xacro="http://ros.org/wiki/xacro">
   <xacro:macro name="asw_eef" params="prefix">
-  <xacro:property name="tcp_cal_filename" value="$(find asw_end_effector)/config/tcp_calibration.yaml"/>
-  <xacro:property name="tcp_cal" value="${load_yaml(tcp_cal_filename)}" />
-  <xacro:property name="eef_mount_offset_filename" value="$(find asw_end_effector)/config/eef_mount_offset.yaml"/>
-  <xacro:property name="eef_mount_offset" value="${load_yaml(eef_mount_offset_filename)}" />
-	<!-- link list -->
-  <link name="${prefix}base_link"/>
-    <visual>
-    	<origin xyz="${eef_mount_offset['transform']['x']} ${eef_mount_offset['transform']['y']} ${eef_mount_offset['transform']['z']}" rpy="0 0 0"/>
-      <geometry>
-        <mesh filename="package://asw_end_effector/meshes/visual/asw_hotend_end_effector.stl" scale=".001 .001 .001"/>
-      </geometry>
-      <material name="grey">
-        <color rgba="0.5 0.5 0.5 1.0"/>
-      </material>
-    </visual>
-    <collision>
-    	<origin xyz="${eef_mount_offset['transform']['x']} ${eef_mount_offset['transform']['y']} ${eef_mount_offset['transform']['z']}" rpy="0 0 0"/>
-      <geometry>
-        <mesh filename="package://asw_end_effector/meshes/collision/asw_hotend_end_effector_shrinked_tip-4mm.stl" scale=".001 .001 .001"/>
-      </geometry>
-      <material name="red">
-        <color rgba="1 0 0 1"/>
-      </material>
-    </collision>
-  </link>
-	<link name="${prefix}tcp_frame"/>
-	<!-- end of link list -->
-	<!-- joint list -->
-  <joint name="${prefix}base_to_tcp" type="fixed">
-		<origin xyz="${tcp_cal['transform']['x']} ${tcp_cal['transform']['y']} ${tcp_cal['transform']['z']}"
-              rpy="${tcp_cal['transform']['roll']} ${tcp_cal['transform']['pitch']} ${tcp_cal['transform']['yaw']}"/>
-    <parent link="${prefix}base_link"/>
-    <child link="${prefix}tcp_frame"/>
-  </joint>
-	<!-- end of joint list -->
-  </xacro:macro>
+		<xacro:property name="tcp_cal_filename" value="$(find asw_end_effector)/config/tcp_calibration.yaml"/>
+		<xacro:property name="tcp_cal" value="${load_yaml(tcp_cal_filename)}" />
+		<xacro:property name="eef_mount_offset_filename" value="$(find asw_end_effector)/config/eef_mount_offset.yaml"/>
+		<xacro:property name="eef_mount_offset" value="${load_yaml(eef_mount_offset_filename)}" />
+		<!-- link list -->
+		<link name="${prefix}base_link">
+		  <visual>
+		  	<origin xyz="${eef_mount_offset['transform']['x']} ${eef_mount_offset['transform']['y']} ${eef_mount_offset['transform']['z']}" rpy="0 0 0"/>
+		    <geometry>
+		      <mesh filename="package://asw_end_effector/meshes/visual/asw_hotend_end_effector.stl" scale=".001 .001 .001"/>
+		    </geometry>
+		    <material name="grey">
+		      <color rgba="0.5 0.5 0.5 1.0"/>
+		    </material>
+		  </visual>
+		  <collision>
+		  	<origin xyz="${eef_mount_offset['transform']['x']} ${eef_mount_offset['transform']['y']} ${eef_mount_offset['transform']['z']}" rpy="0 0 0"/>
+		    <geometry>
+		      <mesh filename="package://asw_end_effector/meshes/collision/asw_hotend_end_effector_shrinked_tip-4mm.stl" scale=".001 .001 .001"/>
+		    </geometry>
+		    <material name="red">
+		      <color rgba="1 0 0 1"/>
+		    </material>
+		  </collision>
+		</link>
+		<link name="${prefix}tcp_frame"/>
+		<!-- end of link list -->
+		<!-- joint list -->
+		<joint name="${prefix}base_to_tcp" type="fixed">
+			<origin xyz="${tcp_cal['transform']['x']} ${tcp_cal['transform']['y']} ${tcp_cal['transform']['z']}"
+		            rpy="${tcp_cal['transform']['roll']} ${tcp_cal['transform']['pitch']} ${tcp_cal['transform']['yaw']}"/>
+		  <parent link="${prefix}base_link"/>
+		  <child link="${prefix}tcp_frame"/>
+		</joint>
+		<!-- end of joint list -->
+	</xacro:macro>
 </robot>

File: framefab_robot/linear_axis/ucla_linear_axis/urdf/ucla_linear_axis_macro.xacro (robot description, xacro)
@@ -2,4 +2,5 @@
 <robot xmlns:xacro="http://ros.org/wiki/xacro">
 	<xacro:property name="half_pi" value="1.5707963267948966"/>
+	<xacro:include filename="$(find ucla_linear_axis)/urdf/resources/materials.xacro"/>
 	<xacro:macro name="ucla_linear_axis" params="prefix">
 	<!--	Link list-->
@@ -7,21 +8,30 @@
 	  <visual>
 		<geometry>
-		  <mesh filename="package://ucla_linear_axis/meshes/visual/ucla_linear_axis_visual_model.stl" scale=".001 .001 .001"/>
+		  <mesh filename="package://ucla_linear_axis/meshes/visual/ucla_linear_axis_visual_rail.stl" scale=".001 .001 .001"/>
 		</geometry>
-		<material name="grey">
-		  <color rgba="0.5 0.5 0.5 1.0"/>
-		</material>
+		<xacro:material_gudel_gray/>
 	  </visual>
 	  <collision>
 		<geometry>
-		  <mesh filename="package://ucla_linear_axis/meshes/collision/ucla_linear_axis_collision_model.stl" scale=".001 .001 .001"/>
+		  <mesh filename="package://ucla_linear_axis/meshes/collision/ucla_linear_axis_collision_rail.stl" scale=".001 .001 .001"/>
 		</geometry>
-		<material name="red">
-		  <color rgba="1 0 0 1"/>
-		</material>
+		<xacro:material_gudel_gray/>
 	  </collision>
 	</link>
 	<link name="${prefix}zero"/>
-	<link name="${prefix}carriage"/>
+  <link name="${prefix}carriage">
+    <visual>
+      <geometry>
+        <mesh filename="package://ucla_linear_axis/meshes/visual/ucla_linear_axis_visual_carriage.stl" scale=".001 .001 .001"/>
+      </geometry>
+			<xacro:material_gudel_green/>
+    </visual>
+    <collision>
+      <geometry>
+        <mesh filename="package://ucla_linear_axis/meshes/collision/ucla_linear_axis_collision_carriage.stl" scale=".001 .001 .001"/>
+      </geometry>
+			<xacro:material_gudel_green/>
+    </collision>
+  </link>
 	<link name="${prefix}robot_mount"/>
 	<!--	End of link list-->
@@ -30,5 +40,5 @@
     <parent link="${prefix}base_link"/>
     <child link="${prefix}zero"/>
-    <origin xyz="$0.0 0.0 0.0" rpy="0 0 0"/>
+    <origin xyz="-3.153 -0.212 0.470" rpy="0 0 0"/>
   </joint>
   <joint name="${prefix}actuation_joint" type="prismatic">
@@ -37,10 +47,10 @@
     <origin xyz="0 0 0" rpy="0 0 0"/>
     <axis xyz="1 0 0"/>
-    <limit lower="-5.750" upper="-0.010" effort="0" velocity="0.150"/>
+    <limit lower="0" upper="5.4" effort="0" velocity="0.150"/>
   </joint>
 	<joint name="${prefix}joint_3" type="fixed">
     <parent link="${prefix}carriage"/>
     <child link="${prefix}robot_mount"/>
-    <origin xyz="0 0 0" rpy="0 0 0"/>
+    <origin xyz="0 0 0.470" rpy="0 0 0"/>
   </joint>
 	<!-- End of joint list -->

Commit message: change eef collision geometry to shrink 6 mm to get passed on topopt-309 small grid.

File: framefab_robot/asw_end_effector/urdf/asw_eef_macro.xacro (robot description, xacro)
@@ -20,5 +20,5 @@
 		  	<origin xyz="${eef_mount_offset['transform']['x']} ${eef_mount_offset['transform']['y']} ${eef_mount_offset['transform']['z']}" rpy="0 0 0"/>
 		    <geometry>
-		      <mesh filename="package://asw_end_effector/meshes/collision/asw_hotend_end_effector_shrinked_tip-4mm.stl" scale=".001 .001 .001"/>
+		      <mesh filename="package://asw_end_effector/meshes/collision/asw_hotend_end_effector_shrinked_tip-6mm.stl" scale=".001 .001 .001"/>
 		    </geometry>
 		    <material name="red">
