Commit message: eth rfl moveit package added.

File: choreo_robot/abb/eth_rfl/eth_rfl_support/urdf/eth_rfl.urdf (robot description, URDF)
Before this commit: robot eth_rfl, 19 links, 18 joints
Links:
- removed link robot_link_cylinder
- removed link robot_link_piston
- link robot_base_link: geometry collision mesh filename=package://abb_irb4400_support/meshes/irb4400l_30_243/collis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; visual mesh filename=package://abb_irb4400_support/meshes/irb4400l_30_243/visual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
- link robot_link_1: geometry collision mesh filename=package://abb_irb4400_support/meshes/irb4400l_30_243/collis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; visual mesh filename=package://abb_irb4400_support/meshes/irb4400l_30_243/visual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
- link robot_link_2: geometry collision mesh filename=package://abb_irb4400_support/meshes/irb4400l_30_243/collis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; visual mesh filename=package://abb_irb4400_support/meshes/irb4400l_30_243/visual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
- link robot_link_3: geometry collision mesh filename=package://abb_irb4400_support/meshes/irb4400l_30_243/collis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; visual mesh filename=package://abb_irb4400_support/meshes/irb4400l_30_243/visual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
- link robot_link_4: geometry collision mesh filename=package://abb_irb4400_support/meshes/irb4400l_30_243/collis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; visual mesh filename=package://abb_irb4400_support/meshes/irb4400l_30_243/visual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
- link robot_link_5: geometry collision mesh filename=package://abb_irb4400_support/meshes/irb4400l_30_243/collis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; visual mesh filename=package://abb_irb4400_support/meshes/irb4400l_30_243/visual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
- link robot_link_6: geometry collision mesh filename=package://abb_irb4400_support/meshes/irb4400l_30_243/collis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; visual mesh filename=package://abb_irb4400_support/meshes/irb4400l_30_243/visual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
Joints:
- removed joint robot_joint_cylinder
- removed joint robot_joint_piston
- joint gantry_to_base_link: origin xyz=1.550 8.675 5.7766 rpy=0 0 0 -> xyz=1.550 0.8675 5.7766 rpy=0 0 0
- joint robot_joint_1: limit lower=-2.967 upper=2.967 effort=0 velocity=1.7453 -> lower=-2.87979 upper=2.87979 effort=0 velocity=2.618; origin xyz=0 0 0.227 rpy=0 0 0 -> xyz=0 0 0 rpy=0 0 0
- joint robot_joint_2: limit lower=-1.134 upper=1.4855 effort=0 velocity=1.5707 -> lower=-1.2217 upper=1.658 effort=0 velocity=2.0944; origin xyz=0.322 0.03 0.551 rpy=0 0 0 -> xyz=0.2 0 0.68 rpy=0 0 0
- joint robot_joint_3: limit lower=-3.142 upper=1.222 effort=0 velocity=1.5707 -> lower=-1.0472 upper=1.1345 effort=0 velocity=2.0944; origin xyz=0 -0.2 1.07 rpy=0 0 0 -> xyz=0 0 0.89 rpy=0 0 0
- joint robot_joint_4: limit lower=-5.236 upper=5.236 effort=0 velocity=2.9671 -> lower=-3.49 upper=3.49 effort=0 velocity=3.927; origin xyz=-0.275 0.181 0.2 rpy=0 0 0 -> xyz=1.38 0 0.15 rpy=0 0 0
- joint robot_joint_5: limit lower=-2.094 upper=2.094 effort=0 velocity=2.4435 -> lower=-2.0944 upper=2.0944 effort=0 velocity=4.3633; origin xyz=1.67 0 0  rpy=0 0 0 -> xyz=0 0 0 rpy=0 0 0
- joint robot_joint_6: limit lower=-6.283 upper=6.283 effort=0 velocity=3.3161 -> lower=-6.9813 upper=6.9813 effort=0 velocity=5.7596; origin xyz=0.153 0 0  rpy=0 0 0 -> xyz=0 0 0 rpy=0 0 0
- joint robot_joint_6-tool0: origin xyz=.055 0 0 rpy=0 1.57079632679 0 -> xyz=0.14 0 0 rpy=0 0 0

File: choreo_robot/abb/eth_rfl/eth_rfl_support/urdf/eth_rfl.xacro (robot description, xacro)
@@ -3,8 +3,8 @@
 	<xacro:property name="half_pi" value="1.5707963267948966"/>
 	<xacro:include filename="$(find eth_rfl_support)/urdf/resources/materials.xacro"/>
-  <xacro:include filename="$(find abb_irb6600_support)/urdf/irb6640_macro.xacro"/>
+  <xacro:include filename="$(find abb_irb4400_support)/urdf/irb4400l_30_243_macro.xacro"/>
 	<xacro:include filename="$(find mit_arch_suction_gripper)/urdf/mit_arch_suction_gripper_macro.xacro"/>
 	<xacro:include filename="$(find eth_rfl_track)/urdf/eth_rfl_track_macro.xacro"/>
-  <xacro:abb_irb6640 prefix="robot_"/>
+  <xacro:abb_irb4400l_30_243 prefix="robot_"/>
   <xacro:suction_gripper prefix="eef_"/>
   <xacro:eth_rfl_track prefix="gantry_"/>
@@ -16,5 +16,5 @@
 	<!--bind the rail to word_frame, can be disabled if using modile platform-->
 	<joint name="gantry_to_base_link" type="fixed">
-    <origin xyz="1.550 8.675 5.7766" rpy="0 0 0"/>
+    <origin xyz="1.550 0.8675 5.7766" rpy="0 0 0"/>
     <parent link="base_link"/>
     <child link="gantry_base_link"/>
