Commit message: add eth_rfl_gripper.

File: choreo_robot/abb/eth_rfl_fixed-xz/eth_rfl_fixed-xz_support/urdf/eth_rfl_fixed-xz.urdf (robot description, URDF)
Before this commit: robot eth_rfl_fixed-xz, 19 links, 18 joints
Links:
- removed link robot_link_cylinder
- removed link robot_link_piston
- added link workspace_base_link
- added link workspace_objects; collision mesh filename=package://eth_rfl_fixed-xz_support/meshes/collision/robarch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 scale=.001 .001 .001; visual mesh filename=package://eth_rfl_fixed-xz_support/meshes/collision/robarch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 scale=.001 .001 .001
- link eef_base_link: geometry collision mesh filename=package://eth_rfl_gripper/meshes/collision/eth_rfl_gripper_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 scale=.001 .001 .001; visual mesh filename=package://eth_rfl_gripper/meshes/visual/eth_rfl_gripper_vis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 scale=.001 .001 .001
- link robot_base_link: geometry collision mesh filename=package://abb_irb4400_support/meshes/irb4400l_30_243/collis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; visual mesh filename=package://abb_irb4400_support/meshes/irb4400l_30_243/visual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
- link robot_link_1: geometry collision mesh filename=package://abb_irb4400_support/meshes/irb4400l_30_243/collis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; visual mesh filename=package://abb_irb4400_support/meshes/irb4400l_30_243/visual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
- link robot_link_2: geometry collision mesh filename=package://abb_irb4400_support/meshes/irb4400l_30_243/collis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; visual mesh filename=package://abb_irb4400_support/meshes/irb4400l_30_243/visual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
- link robot_link_3: geometry collision mesh filename=package://abb_irb4400_support/meshes/irb4400l_30_243/collis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; visual mesh filename=package://abb_irb4400_support/meshes/irb4400l_30_243/visual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
- link robot_link_4: geometry collision mesh filename=package://abb_irb4400_support/meshes/irb4400l_30_243/collis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; visual mesh filename=package://abb_irb4400_support/meshes/irb4400l_30_243/visual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
- link robot_link_5: geometry collision mesh filename=package://abb_irb4400_support/meshes/irb4400l_30_243/collis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; visual mesh filename=package://abb_irb4400_support/meshes/irb4400l_30_243/visual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
- link robot_link_6: geometry collision mesh filename=package://abb_irb4400_support/meshes/irb4400l_30_243/collis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; visual mesh filename=package://abb_irb4400_support/meshes/irb4400l_30_243/visual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
Joints:
- removed joint robot_joint_cylinder
- removed joint robot_joint_piston
- added joint workspace_baselink_to_objects: type fixed, parent workspace_base_link, child workspace_objects, origin xyz=0 0 0 rpy=0 0 0
- added joint world_to_workspace: type fixed, parent base_link, child workspace_base_link, origin xyz=0 0 0 rpy=0 0 0
- joint ee_to_robot: origin xyz=0 0 0 rpy=0 0 0 -> xyz=0 0 0 rpy=0 1.57079632679 0
- joint eef_base_to_tcp: origin xyz=0.145336 0.001949 0.096286 rpy=0.0 1.57079632679 0.0 -> xyz=0.0 0.0 0.475 rpy=1.57079632679 0.0 0.0
- joint gantry_x_joint: origin xyz=0 0 0 rpy=0 0 0 -> xyz=12.173 0 0 rpy=0 0 0
- joint robot_joint_1: limit lower=-2.967 upper=2.967 effort=0 velocity=1.7453 -> lower=-2.87979 upper=2.87979 effort=0 velocity=2.618; origin xyz=0 0 0.780 rpy=0 0 0 -> xyz=0 0 0 rpy=0 0 0
- joint robot_joint_2: limit lower=-1.134 upper=1.4855 effort=0 velocity=1.5707 -> lower=-1.2217 upper=1.658 effort=0 velocity=2.0944; origin xyz=0.320 0 0 rpy=0 0 0 -> xyz=0.2 0 0.68 rpy=0 0 0
- joint robot_joint_3: limit lower=-3.142 upper=1.222 effort=0 velocity=1.5707 -> lower=-1.0472 upper=1.1345 effort=0 velocity=2.0944; origin xyz=0 0 1.075 rpy=0 0 0 -> xyz=0 0 0.89 rpy=0 0 0
- joint robot_joint_4: limit lower=-5.236 upper=5.236 effort=0 velocity=2.9671 -> lower=-3.49 upper=3.49 effort=0 velocity=3.927; origin xyz=0 0 0.2 rpy=0 0 0 -> xyz=1.38 0 0.15 rpy=0 0 0
- joint robot_joint_5: limit lower=-2.094 upper=2.094 effort=0 velocity=2.4435 -> lower=-2.0944 upper=2.0944 effort=0 velocity=4.3633; origin xyz=1.392 0 0  rpy=0 0 0 -> xyz=0 0 0 rpy=0 0 0
- joint robot_joint_6: limit lower=-6.283 upper=6.283 effort=0 velocity=3.3161 -> lower=-6.9813 upper=6.9813 effort=0 velocity=5.7596; origin xyz=0.2 0 0  rpy=0 0 0 -> xyz=0 0 0 rpy=0 0 0
- joint robot_joint_6-tool0: origin xyz=0 0 0 rpy=0 1.57079632679 0 -> xyz=0.14 0 0 rpy=0 0 0

File: choreo_robot/abb/eth_rfl_fixed-xz/eth_rfl_fixed-xz_support/urdf/eth_rfl_fixed-xz.xacro (robot description, xacro)
@@ -3,11 +3,14 @@
 	<xacro:property name="half_pi" value="1.5707963267948966"/>
 	<xacro:include filename="$(find eth_rfl_fixed-xz_support)/urdf/resources/materials.xacro"/>
-  <xacro:include filename="$(find abb_irb6640_support)/urdf/irb6640_185_280_macro.xacro"/>
-	<xacro:include filename="$(find mit_arch_suction_gripper)/urdf/mit_arch_suction_gripper_macro.xacro"/>
+<!--  <xacro:include filename="$(find abb_irb6640_support)/urdf/irb6640_185_280_macro.xacro"/>-->
+  <xacro:include filename="$(find abb_irb4400_support)/urdf/irb4400l_30_243_macro.xacro"/>
+	<xacro:include filename="$(find eth_rfl_gripper)/urdf/eth_rfl_gripper_macro.xacro"/>
 	<xacro:include filename="$(find eth_rfl_fixed-xz_track)/urdf/eth_rfl_fixed-xz_track_macro.xacro"/>
-  <xacro:abb_irb6640_185_280 prefix="robot_"/>
-  <xacro:suction_gripper prefix="eef_"/>
+	<xacro:include filename="$(find eth_rfl_fixed-xz_support)/urdf/robarch_2018_workspace.xacro"/>
+  <xacro:abb_irb4400l_30_243 prefix="robot_"/>
+<!--  <xacro:abb_irb6640_185_280 prefix="robot_"/>-->
+  <xacro:eth_rfl_gripper prefix="eef_"/>
   <xacro:eth_rfl_fixed-xz_track prefix="gantry_"/>
-	<!--  <xacro:simple_linear_track_demo_cell prefix=""/>-->
+	<xacro:robarch_2018_workspace prefix="workspace_"/>
 	<!-- Link list -->
   <link name="base_link"/>
@@ -28,4 +31,9 @@
 		<parent link="robot_tool0"/>
 		<child link="eef_base_link"/>
+		<origin xyz="0 0 0" rpy="0 ${half_pi} 0"/>
+	</joint>
+	<joint name="world_to_workspace" type="fixed">
+		<parent link="base_link"/>
+		<child link="workspace_base_link"/>
 		<origin xyz="0 0 0" rpy="0 0 0"/>
 	</joint>

File: choreo_robot/eth_rfl_fixed-xz_track/urdf/eth_rfl_fixed-xz_track_macro.xacro (robot description, xacro)
@@ -67,5 +67,5 @@
     <parent link="${prefix}base_link"/>
     <child link="${prefix}y_bridge"/>
-    <origin xyz="0 0 0" rpy="0 0 0"/>
+    <origin xyz="12.173 0 0" rpy="0 0 0"/>
   </joint>
   <joint name="${prefix}y_joint" type="prismatic">

Commit message: some tweaks for eth_rfl_fixed_xz demo for robarch 2018.

File: choreo_robot/abb/eth_rfl_fixed-xz/eth_rfl_fixed-xz_support/urdf/eth_rfl_fixed-xz.urdf (robot description, URDF)
Before this commit: robot eth_rfl_fixed-xz, 19 links, 18 joints
Joints:
- joint eef_base_to_tcp: origin xyz=0.0 0.0 0.475 rpy=1.57079632679 0.0 0.0 -> xyz=0.0 0.0 0.475 rpy=1.57079632679 0.0 0
- joint gantry_x_joint: origin xyz=12.173 0 0 rpy=0 0 0 -> xyz=10.5 0 0 rpy=0 0 0
- joint gantry_z_carriage_mount: origin xyz=0.545 -0.0075 -2.526 rpy=0 3.14159265359 0 -> xyz=0.545 -0.0075 -1.2 rpy=0 3.14159265359 0
- joint gantry_z_joint: origin xyz=0 0 0 rpy=0 0 0 -> xyz=0 0 -1 rpy=0 0 0

File: choreo_robot/abb/eth_rfl_fixed-xz/eth_rfl_fixed-xz_support/urdf/robarch_2018_workspace.xacro (robot description, xacro)
@@ -11,7 +11,5 @@
 		<mesh filename="package://eth_rfl_fixed-xz_support/meshes/collision/robarch_2018_workspace_collision.stl" scale=".001 .001 .001"/>
 	</geometry>
-	<material name="grey">
-    	<color rgba="0.5 0.5 0.5 0.9"/>
-	</material>
+	<xacro:material_tan/>
 </visual>
 <collision>

File: choreo_robot/eth_rfl_fixed-xz_track/urdf/eth_rfl_fixed-xz_track_macro.xacro (robot description, xacro)
@@ -67,5 +67,5 @@
     <parent link="${prefix}base_link"/>
     <child link="${prefix}y_bridge"/>
-    <origin xyz="12.173 0 0" rpy="0 0 0"/>
+    <origin xyz="10.5 0 0" rpy="0 0 0"/>
   </joint>
   <joint name="${prefix}y_joint" type="prismatic">
@@ -79,10 +79,10 @@
     <parent link="${prefix}xy_carriage"/>
     <child link="${prefix}z_carriage"/>
-    <origin xyz="0 0 0" rpy="0 0 0"/>
+    <origin xyz="0 0 -1" rpy="0 0 0"/>
   </joint>
 	<joint name="${prefix}z_carriage_mount" type="fixed">
     <parent link="${prefix}z_carriage"/>
     <child link="${prefix}robot_mount"/>
-    <origin xyz="0.545 -0.0075 -2.526" rpy="0 ${2*half_pi} 0"/>
+    <origin xyz="0.545 -0.0075 -1.2" rpy="0 ${2*half_pi} 0"/>
   </joint>
 	<!-- End of joint list -->
