Commit message: take down extrusion head fine geometry model.

File: choreo_robot/asw_end_effector/urdf/asw_eef_macro.xacro (robot description, xacro)
@@ -11,5 +11,5 @@
 		  	<origin xyz="${eef_mount_offset['transform']['x']} ${eef_mount_offset['transform']['y']} ${eef_mount_offset['transform']['z']}" rpy="0 0 0"/>
 		    <geometry>
-		      <mesh filename="package://asw_end_effector/meshes/visual/asw_hotend_end_effector.stl" scale=".001 .001 .001"/>
+		      <mesh filename="package://asw_end_effector/meshes/visual/asw_hotend_end_effector_shrinked_tip-4mm.stl" scale=".001 .001 .001"/>
 		    </geometry>
 		    <material name="grey">

Commit message: add retraction speed. Tweaks for construction robotics video submission.

File: choreo_robot/asw_end_effector/urdf/asw_eef_macro.xacro (robot description, xacro)
@@ -11,5 +11,5 @@
 		  	<origin xyz="${eef_mount_offset['transform']['x']} ${eef_mount_offset['transform']['y']} ${eef_mount_offset['transform']['z']}" rpy="0 0 0"/>
 		    <geometry>
-		      <mesh filename="package://asw_end_effector/meshes/visual/asw_hotend_end_effector_shrinked_tip-4mm.stl" scale=".001 .001 .001"/>
+		      <mesh filename="package://asw_end_effector/meshes/visual/asw_hotend_end_effector.stl" scale=".001 .001 .001"/>
 		    </geometry>
 		    <material name="grey">
